File: mansour_esc_hw/mansour_esc_hw.kicad_pcb (KiCad board)
At the start: 2 copper layers, 55 x 23 mm, 41 parts, among them J1 B+, J2 B-, J3 uC connect, J5 Motor U, J6 Motor V, J7 Motor W, Q1 AON6414A, Q2 AON6414A, Q3 AON6414A, Q4 AON6414A, Q5 AON6414A, Q6 AON6414A, U1 FD6288T

Commit message: adding comments
Other:
- board text added: "at least 2oz copper height(thickness) is required to handle 20A. To reduce cost, go with 1oz copper and pour a lot of solder to GND/Power Zones and motor U/V/W zones. Soldering 2x1mm copper bar on those zones would be great"
Changed lines of the file:
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@@
+		)
+	)
+	(gr_text "at least 2oz copper height(thickness) is required to handle 20A.\nTo reduce cost, go with 1oz copper and\npour a lot of solder to GND/Power Zones and\nmotor U/V/W zones.\nSoldering 2x1mm copper bar on those zones would be great"
+		(at 74.1 30 0)
+		(layer "Cmts.User")
+		(effects
+			(font
+				(size 1 1)
+				(thickness 0.15)
+			)
+			(justify left bottom)
+		)
+	)
+	(dimension
+		(type orthogonal)
+		(layer "Cmts.User")
+		(pts
+			(xy 124.974164 40.05) (xy 124.974164 63.05)
+		)
+		(height 8.225836)
+		(orientation 1)
+		(format
+			(prefix "")
+			(suffix "")
+			(units 3)
+			(units_format 0)
+			(precision 4)
+			(suppress_zeroes yes)
+		)
+		(style
+			(thickness 0.1)
+			(arrow_length 1.27)
+			(text_position_mode 0)
+			(arrow_direction outward)
+			(extension_height 0.58642)
+			(extension_offset 0.5)
+			(keep_text_aligned yes)
+		)
+		(gr_text "23"
+			(at 132.05 51.55 90)
+			(layer "Cmts.User")
+			(effects
+				(font
+					(size 1 1)
+					(thickness 0.15)
+				)
+			)
+		)
+	)
+	(dimension
+		(type orthogonal)
+		(layer "Cmts.User")
+		(pts
+			(xy 69.974164 40.05) (xy 124.974164 40.05)
+		)
+		(height -7.15)
+		(orientation 0)
+		(format
+			(prefix "")
+			(suffix "")
+			(units 3)
+			(units_format 0)
+			(precision 4)
+			(suppress_zeroes yes)
+		)
+		(style
+			(thickness 0.1)
+			(arrow_length 1.27)
+			(text_position_mode 0)
+			(arrow_direction outward)
+			(extension_height 0.58642)
+			(extension_offset 0.5)
+			(keep_text_aligned yes)
+		)
+		(gr_text "55"
+			(at 97.474164 31.75 0)
+			(layer "Cmts.User")
+			(effects
+				(font
+					(size 1 1)
+					(thickness 0.15)
+				)
+			)
 		)
 	)
